File: VoltRefBoard.sch (EAGLE design)
At the start: 29 parts, among them J1 BANANA_CONN, J2 BANANA_CONN, J3 BANANA_CONN, J4 BANANA_CONN, J5 BANANA_CONN, U1 MAX6225ACSA+, U2 MAX6250ACSA+

Commit message: Latest commits
Parts:
- LED1: MF (none) -> OSRAM; MPN (none) -> LGT67K-H2K1-24-Z; OC_FARNELL unknown -> 1226376
- TM1, TM2: MF (none) -> VISHAY SFERNICE; MPN (none) -> TS53YJ103MR10; OC_FARNELL unknown -> 1141485
- TP1, TP2, TP3: MF (none) -> MULTICOMP; MPN (none) -> TEST-3; OC_FARNELL unknown -> 1702006
Other:
- note added: "Banana plug socket holes may not be the right size. Also need to be different colours"
Changed lines of the file:
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@@
 </part>
 <part name="TP1" library="TP_1MM_TH" deviceset="TP_1MM_TH" device="&quot;">
-<attribute name="MF" value=""/>
-<attribute name="MPN" value=""/>
-<attribute name="OC_FARNELL" value="unknown"/>
+<attribute name="MF" value="MULTICOMP"/>
+<attribute name="MPN" value="TEST-3"/>
+<attribute name="OC_FARNELL" value="1702006"/>
 </part>
 <part name="TP3" library="TP_1MM_TH" deviceset="TP_1MM_TH" device="&quot;">
-<attribute name="MF" value=""/>
-<attribute name="MPN" value=""/>
-<attribute name="OC_FARNELL" value="unknown"/>
+<attribute name="MF" value="MULTICOMP"/>
+<attribute name="MPN" value="TEST-3"/>
+<attribute name="OC_FARNELL" value="1702006"/>
 </part>
 <part name="SUPPLY13" library="supply2" deviceset="GND" device=""/>
@@
 </part>
 <part name="TP2" library="TP_1MM_TH" deviceset="TP_1MM_TH" device="&quot;">
-<attribute name="MF" value=""/>
-<attribute name="MPN" value=""/>
-<attribute name="OC_FARNELL" value="unknown"/>
+<attribute name="MF" value="MULTICOMP"/>
+<attribute name="MPN" value="TEST-3"/>
+<attribute name="OC_FARNELL" value="1702006"/>
 </part>
 <part name="SUPPLY1" library="supply2" deviceset="GND" device=""/>
@@
 </part>
 <part name="LED1" library="P-LCC-2_Shorter" deviceset="LED" device="P-LCC-2" value="GREEN_LED">
-<attribute name="MF" value=""/>
-<attribute name="MPN" value=""/>
-<attribute name="OC_FARNELL" value="unknown"/>
+<attribute name="MF" value="OSRAM"/>
+<attribute name="MPN" value="LGT67K-H2K1-24-Z"/>
+<attribute name="OC_FARNELL" value="1226376"/>
 </part>
 <part name="R1" library="rcl" deviceset="R-EU_" device="R0805" value="2k">
@@
 </part>
 <part name="TM1" library="P-LCC-2_Shorter" deviceset="TRIMPOT" device="TC33X" value="10k">
-<attribute name="MF" value=""/>
-<attribute name="MPN" value=""/>
-<attribute name="OC_FARNELL" value="unknown"/>
+<attribute name="MF" value="VISHAY SFERNICE"/>
+<attribute name="MPN" value="TS53YJ103MR10"/>
+<attribute name="OC_FARNELL" value="1141485"/>
 </part>
 <part name="TM2" library="P-LCC-2_Shorter" deviceset="TRIMPOT" device="TC33X" value="10k">
-<attribute name="MF" value=""/>
-<attribute name="MPN" value=""/>
-<attribute name="OC_FARNELL" value="unknown"/>
+<attribute name="MF" value="VISHAY SFERNICE"/>
+<attribute name="MPN" value="TS53YJ103MR10"/>
+<attribute name="OC_FARNELL" value="1141485"/>
 </part>
 <part name="F1" library="adafruit" deviceset="PTCFUSE" device="-1812" value="1.1A">
@@
 <text x="-55.88" y="7.62" size="1.778" layer="91">ON/OFF/ON</text>
 <text x="43.18" y="45.72" size="3.81" layer="91">WWW.GUVVY.CO.UK</text>
+<text x="149.86" y="50.8" size="1.778" layer="91">Banana plug socket holes may not be the right size. Also need to be different colours</text>
 </plain>
 <instances>

Commit message: Added the 5x5 pcbs from sick of beige
Added the 5x5 pcbs from sick of beige and added cost down notes to the
schematic to make it cheap to manufacture
Parts:
- removed PAD1, PAD2, PAD3, PAD4: MOUNT_HOLE, wirepad:3,81/1,4
- added PCB1: PCB_DP_SQUARE-5X5, dp_devices:PCB_DP_SQUARE-5X5
- added U$1, U$2, U$3, U$4: FIDUCIAL, adafruit:FIDUCIAL
Connections:
- net GND: no longer PAD1.P, PAD2.P, PAD3.P, PAD4.P
Other:
- note added: "CHANGE: - input 4mm to screw terminals. - battery terminal can be removed, just provide 2 x 9v batteries to attach to the - Potentiometer to a cermet device - Re-arrange for one 10v device with pot down for other voltages - Consider replacing output terminals with just test points, just having input voltage terminals. - Work out if an input bridge rectifier is cheaper than fuse+diode. - Make it a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"
Changed lines of the file:
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@@
 <?xml version="1.0" encoding="utf-8"?>
 <!DOCTYPE eagle SYSTEM "eagle.dtd">
-<eagle version="6.5.0">
+<eagle version="7.5.0">
 <drawing>
 <settings>
@@
 <part name="SUPPLY1" library="supply2" deviceset="GND" device=""/>
 <part name="SUPPLY2" library="supply2" deviceset="GND" device=""/>
-<part name="PAD1" library="wirepad" deviceset="3,81/1,4" device="" value="MOUNT_HOLE">
-<attribute name="MF" value=""/>
-<attribute name="MPN" value=""/>
-<attribute name="OC_FARNELL" value="unknown"/>
-</part>
-<part name="PAD2" library="wirepad" deviceset="3,81/1,4" device="" value="MOUNT_HOLE">
-<attribute name="MF" value=""/>
-<attribute name="MPN" value=""/>
-<attribute name="OC_FARNELL" value="unknown"/>
-</part>
-<part name="PAD3" library="wirepad" deviceset="3,81/1,4" device="" value="MOUNT_HOLE">
-<attribute name="MF" value=""/>
-<attribute name="MPN" value=""/>
-<attribute name="OC_FARNELL" value="unknown"/>
-</part>
-<part name="PAD4" library="wirepad" deviceset="3,81/1,4" device="" value="MOUNT_HOLE">
-<attribute name="MF" value=""/>
-<attribute name="MPN" value=""/>
-<attribute name="OC_FARNELL" value="unknown"/>
-</part>
 <part name="LOGO1" library="SparkFun-Aesthetics" deviceset="OSHW-LOGO" device="L">
 <attribute name="MF" value=""/>
@@
 </part>
 <part name="SUPPLY3" library="supply2" deviceset="GND" device=""/>
+<part name="PCB1" library="dp_devices" deviceset="PCB_DP_SQUARE" device="-5X5"/>
+<part name="U$1" library="adafruit" deviceset="FIDUCIAL" device=""/>
+<part name="U$2" library="adafruit" deviceset="FIDUCIAL" device=""/>
+<part name="U$3" library="adafruit" deviceset="FIDUCIAL" device=""/>
+<part name="U$4" library="adafruit" deviceset="FIDUCIAL" device=""/>
 </parts>
 <sheets>
@@
 <text x="43.18" y="45.72" size="3.81" layer="91">WWW.GUVVY.CO.UK</text>
 <text x="149.86" y="50.8" size="1.778" layer="91">Banana plug socket holes may not be the right size. Also need to be different colours</text>
+<text x="-137.16" y="114.3" size="5.08" layer="91">CHANGE:
+- input 4mm to screw terminals.
+- battery terminal can be removed, just provide 2 x 9v batteries to attach to the
+- Potentiometer to a cermet device
+- Re-arrange for one 10v device with pot down for other voltages
+- Consider replacing output terminals with just test points, just having input voltage terminals.
+- Work out if an input bridge rectifier is cheaper than fuse+diode.
+- Make it all SMD, especially the switch, infact does it need a switch?
+- Add resistors and options for cap / inductors</text>
 </plain>
 <instances>
@@
 <instance part="SUPPLY1" gate="GND" x="236.22" y="-38.1"/>
 <instance part="SUPPLY2" gate="GND" x="-81.28" y="-45.72"/>
-<instance part="PAD1" gate="1" x="254" y="-2.54" rot="R180">
-<attribute name="OC_FARNELL" x="254" y="-2.54" size="1.778" layer="96" rot="R90" display="off"/>
-<attribute name="MF" x="254" y="-2.54" size="1.778" layer="96" rot="R90" display="off"/>
-<attribute name="MPN" x="254" y="-2.54" size="1.778" layer="96" rot="R90" display="off"/>
-</instance>
-<instance part="PAD2" gate="1" x="254" y="-10.16" rot="R180">
-<attribute name="OC_FARNELL" x="254" y="-10.16" size="1.778" layer="96" rot="R90" display="off"/>
-<attribute name="MF" x="254" y="-10.16" size="1.778" layer="96" rot="R90" display="off"/>
-<attribute name="MPN" x="254" y="-10.16" size="1.778" layer="96" rot="R90" display="off"/>
-</instance>
-<instance part="PAD3" gate="1" x="254" y="-17.78" rot="R180">
-<attribute name="OC_FARNELL" x="254" y="-17.78" size="1.778" layer="96" rot="R90" display="off"/>
-<attribute name="MF" x="254" y="-17.78" size="1.778" layer="96" rot="R90" display="off"/>
-<attribute name="MPN" x="254" y="-17.78" size="1.778" layer="96" rot="R90" display="off"/>
-</instance>
-<instance part="PAD4" gate="1" x="254" y="-25.4" rot="R180">
-<attribute name="OC_FARNELL" x="254" y="-25.4" size="1.778" layer="96" rot="R90" display="off"/>
-<attribute name="MF" x="254" y="-25.4" size="1.778" layer="96" rot="R90" display="off"/>
-<attribute name="MPN" x="254" y="-25.4" size="1.778" layer="96" rot="R90" display="off"/>
-</instance>
 <instance part="LOGO1" gate="G$1" x="68.58" y="66.04">
 <attribute name="OC_FARNELL" x="68.58" y="66.04" size="1.778" layer="96" rot="R90" display="off"/>
@@
 </instance>
 <instance part="SUPPLY3" gate="GND" x="-5.08" y="0"/>
+<instance part="PCB1" gate="PCB" x="68.58" y="104.14"/>
+<instance part="U$1" gate="G$1" x="48.26" y="88.9"/>
+<instance part="U$2" gate="G$1" x="58.42" y="88.9"/>
+<instance part="U$3" gate="G$1" x="68.58" y="88.9"/>
+<instance part="U$4" gate="G$1" x="78.74" y="88.9"/>
 </instances>
 <busses>
@@
 <wire x1="251.46" y1="30.48" x2="243.84" y2="30.48" width="0.1524" layer="91"/>
 <wire x1="243.84" y1="30.48" x2="236.22" y2="30.48" width="0.1524" layer="91"/>
-<pinref part="PAD4" gate="1" pin="P"/>
-<wire x1="236.22" y1="-2.54" x2="236.22" y2="-10.16" width="0.1524" layer="91"/>
-<wire x1="236.22" y1="-10.16" x2="236.22" y2="-17.78" width="0.1524" layer="91"/>
-<wire x1="236.22" y1="-17.78" x2="236.22" y2="-25.4" width="0.1524" layer="91"/>
-<wire x1="236.22" y1="-25.4" x2="251.46" y2="-25.4" width="0.1524" layer="91"/>
-<pinref part="PAD3" gate="1" pin="P"/>
-<wire x1="251.46" y1="-17.78" x2="236.22" y2="-17.78" width="0.1524" layer="91"/>
-<junction x="236.22" y="-17.78"/>
-<pinref part="PAD2" gate="1" pin="P"/>
-<wire x1="251.46" y1="-10.16" x2="236.22" y2="-10.16" width="0.1524" layer="91"/>
-<junction x="236.22" y="-10.16"/>
-<pinref part="PAD1" gate="1" pin="P"/>
-<wire x1="251.46" y1="-2.54" x2="236.22" y2="-2.54" width="0.1524" layer="91"/>
-<junction x="236.22" y="-2.54"/>
-<wire x1="236.22" y1="30.48" x2="236.22" y2="-2.54" width="0.1524" layer="91"/>
 <pinref part="SUPPLY1" gate="GND" pin="GND"/>
-<wire x1="236.22" y1="-35.56" x2="236.22" y2="-25.4" width="0.1524" layer="91"/>
-<junction x="236.22" y="-25.4"/>
+<wire x1="236.22" y1="-35.56" x2="236.22" y2="30.48" width="0.1524" layer="91"/>
 <pinref part="TP3" gate="G$1" pin="1"/>
 <junction x="243.84" y="30.48"/>

Commit message: adding latest updates
adding latest updates
Parts:
- removed BAT1: +9V_BATTERY, BC9VPC_ShortenedSilkScreen:BC9VPC
- removed D1: MBR60H100CTG, diode:DIODE-2AC|CATO220V
- removed J4, J5: BANANA_CONN, SparkFun-Connectors:BANANA_CONN
- added D2: (no value), adafruit:DIODESOD-323F
- added J6: 1X2-3.5MM, adafruit:1X2-3.5MM
- added TP4: TP_1MM_TH", TP_1MM_TH:TP_1MM_TH"
- F1: value 1.1A -> PTC_0805_100MA; device adafruit:PTCFUSE-1812 -> rcl:R-EU_R0805
- J1, J2: value BANANA_CONN -> 1X2-3.5MM; device SparkFun-Connectors:BANANA_CONN -> adafruit:1X2-3.5MM
- J3: value BANANA_CONN -> 2060-402; device SparkFun-Connectors:BANANA_CONN -> Wago-2060-402:2060-402; OC_FARNELL unknown -> (none)
- PCB1, U$1, U$2, U$3, U$4: OC_FARNELL (none) -> unknown
- S1: value 5649A -> (none); device Switch_320-938_Corrected:320-938 -> SparkFun-Electromechanical:SWITCH-SPDT-SMD-A; MF APEM -> (none); MPN 5649A -> (none); OC_FARNELL 1082316 -> unknown
- U1: MPN (none) -> MAX6225ACSA+.
- U2: MPN (none) -> MAX6250ACSA+.
Connections:
- removed net V_IN_B: BAT1.V+, S11.O, S1B.O
- net +2.5V_REF: now also J1.1; no longer J3.1
- net +5.0V_REF: now also J2.1; no longer J4.1
- net GND: now also D2.A, J1.2, J2.2, J6.2, TP4.1; no longer BAT1.V-, D1.A1, D1.A2, J2.1, J5.1
- net V_IN_0: now also S1.P; no longer S11.P, S1B.P
- net V_IN_1: now also D2.C; no longer D1.C
- net V_IN_A: now also J6.1, S1.S; no longer J1.1, S11.S, S1B.S
Other:
- note added: "CONSIDER USING THE WAGO SMD PUSH BUTTON CONNECTOR INSTEAD OF TH CONNECTOR"
- note added: "ON/OFF"
- note removed: "ON/OFF/ON"
- moved on the sheet: TP3

Commit message: minor updates
Parts:
- removed J3: 2060-402, Wago-2060-402:2060-402
Other:
- note removed: "CONSIDER USING THE WAGO SMD PUSH BUTTON CONNECTOR INSTEAD OF TH CONNECTOR"
Changed lines of the file:
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@@
 <attribute name="OC_FARNELL" value="1757770"/>
 </part>
-<part name="J3" library="Wago-2060-402" deviceset="2060-402" device=""/>
 </parts>
 <sheets>
@@
 - Make it all SMD, especially the switch, infact does it need a switch?
 - Add resistors and options for cap / inductors</text>
-<text x="-86.36" y="-15.24" size="1.778" layer="91">CONSIDER USING THE WAGO SMD PUSH BUTTON CONNECTOR INSTEAD OF TH CONNECTOR</text>
 </plain>
 <instances>
@@
 <attribute name="MPN" x="-5.08" y="22.86" size="1.778" layer="96" display="off"/>
 </instance>
-<instance part="J3" gate="A" x="-99.06" y="-12.7"/>
 </instances>
 <busses>
